File: clock_schematic_and_layout/clock_schematic_and_layout.kicad_pcb (KiCad board)
At the start: 2 copper layers, 48 parts, among them U1 ATmega16A-PU, X1 SG-8002CA

Commit message: Finished schematic and PCB layout. Haven't properly double checked the schematic though :'( (can't be bothered haha.)
Parts:
- removed REF**: DSUB-9_Female_Horizontal_P2.77x2.84mm_EdgePinOffset7.70mm_H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, Connector_Dsub:DSUB-9_Female_Horizontal_P2.77x2.84mm_EdgePinOffset7.70mm_Housed_MountingHolesOffset9.12mm
- removed REF** (x18): LED_D3.0mm_Horizontal_O1.27mm_Z2.0mm_Clear, LED_THT:LED_D3.0mm_Horizontal_O1.27mm_Z2.0mm_Clear
- removed REF** (x18): R_Axial_DIN0207_L6.3mm_D2.5mm_P7.62mm_Horizontal, Resistor_THT:R_Axial_DIN0207_L6.3mm_D2.5mm_P7.62mm_Horizontal
- removed REF**: Crystal_SMD_TXC_9HT11-2Pin_2.0x1.2mm_HandSoldering, Crystal:Crystal_SMD_TXC_9HT11-2Pin_2.0x1.2mm_HandSoldering
- removed REF** (x3): CP_Radial_D4.0mm_P2.00mm, Capacitor_THT:CP_Radial_D4.0mm_P2.00mm
- removed REF**: D_MELF-RM10_Universal_Handsoldering, Diode_SMD:D_MELF-RM10_Universal_Handsoldering
- removed REF** (x3): DIP-16_W7.62mm_LongPads, Package_DIP:DIP-16_W7.62mm_LongPads
- removed REF**: TSOT-23-5_HandSoldering, Package_TO_SOT_SMD:TSOT-23-5_HandSoldering
- added AH1: LED, LED_THT:LED_D3.0mm_Horizontal_O1.27mm_Z2.0mm_Clear, F.Cu at (57.4, 94.7)
- added AM1: LED, LED_THT:LED_D3.0mm_Horizontal_O1.27mm_Z2.0mm_Clear, F.Cu at (76.5, 94.7)
- added AS1: LED, LED_THT:LED_D3.0mm_Horizontal_O1.27mm_Z2.0mm_Clear, F.Cu at (95.5, 94.7)
- added C1: 0.01uF, Crystal:Crystal_SMD_TXC_9HT11-2Pin_2.0x1.2mm_HandSoldering, F.Cu at (111.3, 88.1)
- added C2: 1uF, Capacitor_THT:CP_Radial_D4.0mm_P2.00mm, F.Cu at (120.9, 75.2)
- added C3: byp, Capacitor_THT:CP_Radial_D4.0mm_P2.00mm, F.Cu at (112.8, 83.6)
- added C4: 1uF, Capacitor_THT:CP_Radial_D4.0mm_P2.00mm, F.Cu at (112.8, 75.2)
- added CD74HC390E1: CD74HC390E, Package_DIP:DIP-16_W7.62mm_LongPads, F.Cu at (136.4, 20.1)
- added CD74HC390E2: CD74HC390E, Package_DIP:DIP-16_W7.62mm_LongPads, F.Cu at (136.4, 42.9)
- added CD74HC390E3: CD74HC390E, Package_DIP:DIP-16_W7.62mm_LongPads, F.Cu at (133.6, 99.6)
- added CLK1: LED, LED_THT:LED_D3.0mm_Horizontal_O1.27mm_Z2.0mm_Clear, F.Cu at (57.4, 24.6)
- added D1: DIODE, Diode_SMD:D_MELF-RM10_Universal_Handsoldering, F.Cu at (110.3, 99.4)
- added H1: LED, LED_THT:LED_D3.0mm_Horizontal_O1.27mm_Z2.0mm_Clear, F.Cu at (57.4, 36.3)
- added H2: LED, LED_THT:LED_D3.0mm_Horizontal_O1.27mm_Z2.0mm_Clear, F.Cu at (57.4, 48.0)
- added H3: LED, LED_THT:LED_D3.0mm_Horizontal_O1.27mm_Z2.0mm_Clear, F.Cu at (57.4, 59.7)
- added H4: LED, LED_THT:LED_D3.0mm_Horizontal_O1.27mm_Z2.0mm_Clear, F.Cu at (57.4, 71.4)
- added H5: LED, LED_THT:LED_D3.0mm_Horizontal_O1.27mm_Z2.0mm_Clear, F.Cu at (57.4, 83.1)
- added J1: DB9_Male, Connector_Dsub:DSUB-9_Female_Horizontal_P2.77x2.84mm_EdgePinOffset7.70mm_Housed_MountingHolesOffset9.12mm, F.Cu at (139.5, 79.5)
- added L1: LDK130M32R, Package_TO_SOT_SMD:TSOT-23-5_HandSoldering, F.Cu at (119.2, 83.5)
- added M1: LED, LED_THT:LED_D3.0mm_Horizontal_O1.27mm_Z2.0mm_Clear, F.Cu at (76.5, 24.6)
- added M2: LED, LED_THT:LED_D3.0mm_Horizontal_O1.27mm_Z2.0mm_Clear, F.Cu at (76.5, 36.3)
- added M3: LED, LED_THT:LED_D3.0mm_Horizontal_O1.27mm_Z2.0mm_Clear, F.Cu at (76.5, 48.0)
- added M4: LED, LED_THT:LED_D3.0mm_Horizontal_O1.27mm_Z2.0mm_Clear, F.Cu at (76.5, 59.7)
- added M5: LED, LED_THT:LED_D3.0mm_Horizontal_O1.27mm_Z2.0mm_Clear, F.Cu at (76.5, 71.4)
- added M6: LED, LED_THT:LED_D3.0mm_Horizontal_O1.27mm_Z2.0mm_Clear, F.Cu at (76.5, 83.1)
- added RAH1: R330, Resistor_THT:R_Axial_DIN0207_L6.3mm_D2.5mm_P7.62mm_Horizontal, F.Cu at (62.5, 89.7)
- added RAM1: R330, Resistor_THT:R_Axial_DIN0207_L6.3mm_D2.5mm_P7.62mm_Horizontal, F.Cu at (81.6, 89.7)
- added RAS1: R330, Resistor_THT:R_Axial_DIN0207_L6.3mm_D2.5mm_P7.62mm_Horizontal, F.Cu at (100.9, 89.7)
- added RCLK1: R330, Resistor_THT:R_Axial_DIN0207_L6.3mm_D2.5mm_P7.62mm_Horizontal, F.Cu at (62.5, 19.6)
- added RH1: R330, Resistor_THT:R_Axial_DIN0207_L6.3mm_D2.5mm_P7.62mm_Horizontal, F.Cu at (62.5, 31.2)
- added RH2: R330, Resistor_THT:R_Axial_DIN0207_L6.3mm_D2.5mm_P7.62mm_Horizontal, F.Cu at (62.5, 42.9)
- added RH3: R330, Resistor_THT:R_Axial_DIN0207_L6.3mm_D2.5mm_P7.62mm_Horizontal, F.Cu at (62.5, 54.6)
- added RH4: R330, Resistor_THT:R_Axial_DIN0207_L6.3mm_D2.5mm_P7.62mm_Horizontal, F.Cu at (62.5, 66.3)
- added RH5: R330, Resistor_THT:R_Axial_DIN0207_L6.3mm_D2.5mm_P7.62mm_Horizontal, F.Cu at (62.5, 78.0)
- added RM1: R330, Resistor_THT:R_Axial_DIN0207_L6.3mm_D2.5mm_P7.62mm_Horizontal, F.Cu at (81.6, 19.6)
- added RM2: R330, Resistor_THT:R_Axial_DIN0207_L6.3mm_D2.5mm_P7.62mm_Horizontal, F.Cu at (81.6, 31.2)
- added RM3: R330, Resistor_THT:R_Axial_DIN0207_L6.3mm_D2.5mm_P7.62mm_Horizontal, F.Cu at (81.6, 42.9)
- added RM4: R330, Resistor_THT:R_Axial_DIN0207_L6.3mm_D2.5mm_P7.62mm_Horizontal, F.Cu at (81.6, 54.6)
- added RM5: R330, Resistor_THT:R_Axial_DIN0207_L6.3mm_D2.5mm_P7.62mm_Horizontal, F.Cu at (81.6, 66.3)
- added RM6: R330, Resistor_THT:R_Axial_DIN0207_L6.3mm_D2.5mm_P7.62mm_Horizontal, F.Cu at (81.6, 78.0)
- added RS1: R330, Resistor_THT:R_Axial_DIN0207_L6.3mm_D2.5mm_P7.62mm_Horizontal, F.Cu at (100.9, 19.6)
- added RS2: R330, Resistor_THT:R_Axial_DIN0207_L6.3mm_D2.5mm_P7.62mm_Horizontal, F.Cu at (100.9, 31.2)
- added RS3: R330, Resistor_THT:R_Axial_DIN0207_L6.3mm_D2.5mm_P7.62mm_Horizontal, F.Cu at (100.9, 42.9)
- added RS4: R330, Resistor_THT:R_Axial_DIN0207_L6.3mm_D2.5mm_P7.62mm_Horizontal, F.Cu at (100.9, 54.6)
- added RS5: R330, Resistor_THT:R_Axial_DIN0207_L6.3mm_D2.5mm_P7.62mm_Horizontal, F.Cu at (100.9, 66.3)
- added RS6: R330, Resistor_THT:R_Axial_DIN0207_L6.3mm_D2.5mm_P7.62mm_Horizontal, F.Cu at (100.9, 78.0)
- added S1: LED, LED_THT:LED_D3.0mm_Horizontal_O1.27mm_Z2.0mm_Clear, F.Cu at (95.5, 24.6)
- added S2: LED, LED_THT:LED_D3.0mm_Horizontal_O1.27mm_Z2.0mm_Clear, F.Cu at (95.5, 36.3)
- added S3: LED, LED_THT:LED_D3.0mm_Horizontal_O1.27mm_Z2.0mm_Clear, F.Cu at (95.5, 48.0)
- added S4: LED, LED_THT:LED_D3.0mm_Horizontal_O1.27mm_Z2.0mm_Clear, F.Cu at (95.5, 59.7)
- added S5: LED, LED_THT:LED_D3.0mm_Horizontal_O1.27mm_Z2.0mm_Clear, F.Cu at (95.5, 71.4)
- added S6: LED, LED_THT:LED_D3.0mm_Horizontal_O1.27mm_Z2.0mm_Clear, F.Cu at (95.5, 83.1)
- X1: footprint Oscillator:Oscillator_SMD_SeikoEpson_SG8002CA-4Pin_7.0x5.0mm -> Oscillator:Oscillator_SMD_SeikoEpson_SG8002CA-4Pin_7.0x5.0mm_HandSoldering
- moved U1 56.4 mm to (125.8, 68.3), turned to 180 degrees
- moved X1 34.3 mm to (117.9, 89.9), turned to -90 degrees
Routing:
- net /GND_(0V): track 0.00 -> 737.8 mm, vias 0 -> 10
- net Net-(CD74HC390E1-Pad3): track 0.00 -> 164.5 mm, vias 0 -> 3
- net Net-(J1-Pad9): track 0.00 -> 164.1 mm, vias 0 -> 1
- net Net-(C4-Pad2): track 0.00 -> 150.7 mm, vias 0 -> 4
- net Net-(CD74HC390E1-Pad14): track 0.00 -> 132.3 mm, vias 0 -> 4
- net Net-(RH1-Pad1): track 0.00 -> 125.2 mm
- net Net-(RH2-Pad1): track 0.00 -> 116.1 mm
- net Net-(RH3-Pad1): track 0.00 -> 109.5 mm
- net Net-(RH4-Pad1): track 0.00 -> 102.4 mm
- net Net-(RM6-Pad1): track 0.00 -> 102.1 mm
- net Net-(RAH1-Pad1): track 0.00 -> 95.8 mm
- net Net-(RH5-Pad1): track 0.00 -> 89.7 mm
- net Net-(RM5-Pad1): track 0.00 -> 82.8 mm
- net Net-(RS6-Pad1): track 0.00 -> 74.9 mm
- net (no net): track 72.1 -> 0.00 mm
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- added copper zone on B.Cu, net /GND_(0V)
- added copper zone on F.Cu, net /GND_(0V)
Other:
- board outline added: 118.4 x 87.6 mm
